Commit message: fixed error "The group 'UR_arm' is not a chain" base_link had 2 childs (base_link_inertia+base)

File: mur/mur_moveit_config/config/mur.srdf.xacro (robot description, xacro)
@@ -13,5 +13,5 @@
     <!--SUBGROUPS: Groups can also be formed by referencing to already defined group names-->
     <group name="UR_arm">
-        <joint name="$(arg prefix)base_link-base_fixed_joint"/>
+        <!-- <joint name="$(arg prefix)base_link-base_fixed_joint"/> -->
         <joint name="$(arg prefix)base_link-base_link_inertia"/>
         <joint name="$(arg prefix)shoulder_pan_joint"/>

Commit message: removed flange-tool from UR-arm group (moveit)

File: mur/mur_moveit_config/config/mur.srdf.xacro (robot description, xacro)
@@ -21,6 +21,6 @@
         <joint name="$(arg prefix)wrist_2_joint"/>
         <joint name="$(arg prefix)wrist_3_joint"/>
-        <joint name="$(arg prefix)wrist_3-flange"/>
-        <joint name="$(arg prefix)flange-tool0"/>
+        <!-- <joint name="$(arg prefix)wrist_3-flange"/>
+        <joint name="$(arg prefix)flange-tool0"/> -->
     </group>
     <!--GROUP STATES: Purpose: Define a named state for a particular group, in terms of joint values. This is useful to define states like 'folded arms'-->
