Commit message: added folded_down poses for both urs

File: mur/mur_moveit_config/config/mur620.srdf.xacro (robot description, xacro)
@@ -202,4 +202,20 @@
         <joint name="$(arg prefix)_r/wrist_1_joint" value="-1.7009"/>
         <joint name="$(arg prefix)_r/wrist_2_joint" value="-1.5621"/>
+        <joint name="$(arg prefix)_r/wrist_3_joint" value="0"/>
+    </group_state>
+    <group_state name="folded_down" group="UR_arm_r">
+        <joint name="$(arg prefix)_r/elbow_joint" value="3.14159265359"/>
+        <joint name="$(arg prefix)_r/shoulder_lift_joint" value="-3.14159265359"/>
+        <joint name="$(arg prefix)_r/shoulder_pan_joint" value="0.0"/>
+        <joint name="$(arg prefix)_r/wrist_1_joint" value="-1.57079632679"/>
+        <joint name="$(arg prefix)_r/wrist_2_joint" value="3.14159265359"/>
+        <joint name="$(arg prefix)_r/wrist_3_joint" value="0"/>
+    </group_state>
+    <group_state name="folded_down" group="UR_arm_l">
+        <joint name="$(arg prefix)_r/elbow_joint" value="0.0"/>
+        <joint name="$(arg prefix)_r/shoulder_lift_joint" value="-3.14159265359"/>
+        <joint name="$(arg prefix)_r/shoulder_pan_joint" value="0.0"/>
+        <joint name="$(arg prefix)_r/wrist_1_joint" value="-1.57079632679"/>
+        <joint name="$(arg prefix)_r/wrist_2_joint" value="3.14159265359"/>
         <joint name="$(arg prefix)_r/wrist_3_joint" value="0"/>
     </group_state>

Commit message: work in progress

File: mur/mur_moveit_config/config/mur620.srdf.xacro (robot description, xacro)
@@ -213,10 +213,10 @@
     </group_state>
     <group_state name="folded_down" group="UR_arm_l">
-        <joint name="$(arg prefix)_r/elbow_joint" value="0.0"/>
-        <joint name="$(arg prefix)_r/shoulder_lift_joint" value="-3.14159265359"/>
-        <joint name="$(arg prefix)_r/shoulder_pan_joint" value="0.0"/>
-        <joint name="$(arg prefix)_r/wrist_1_joint" value="-1.57079632679"/>
-        <joint name="$(arg prefix)_r/wrist_2_joint" value="3.14159265359"/>
-        <joint name="$(arg prefix)_r/wrist_3_joint" value="0"/>
+        <joint name="$(arg prefix)_l/elbow_joint" value="0.0"/>
+        <joint name="$(arg prefix)_l/shoulder_lift_joint" value="-3.14159265359"/>
+        <joint name="$(arg prefix)_l/shoulder_pan_joint" value="0.0"/>
+        <joint name="$(arg prefix)_l/wrist_1_joint" value="-1.57079632679"/>
+        <joint name="$(arg prefix)_l/wrist_2_joint" value="3.14159265359"/>
+        <joint name="$(arg prefix)_l/wrist_3_joint" value="0"/>
     </group_state>
     <!--END EFFECTOR: Purpose: Represent information about an end effector.-->
