Commit message: Add keyence_lj_x.urdf.xacro for simulation

File: mur/mur_description/urdf/mur_620.gazebo.xacro (robot description, xacro)
@@ -30,4 +30,5 @@
 	<xacro:if value="${sim}">
 		<xacro:include filename="$(find schunk_emh_rp_45)/urdf/schunk_emh_rp_045.urdf.xacro"/>
+		<xacro:include filename="$(find keyence_lj_x)/urdf/keyence_lj_x.urdf.xacro"/>
 	</xacro:if>
 	<!-- Init the MiR200 marco that is also used for the hardware -->
@@ -85,29 +86,9 @@
 		<xacro:schunk_emh_rp_045 tf_prefix="UR10_r"	tool_link="UR10_r/flange"/>
 		<xacro:schunk_emh_rp_045 tf_prefix="UR10_l"	tool_link="UR10_l/flange"/>
+		<xacro:keyence_lj_x tf_prefix="UR10_r"	tool_link="UR10_r/flange"/>
+		<xacro:keyence_lj_x tf_prefix="UR10_l"	tool_link="UR10_l/flange"/>
 	</xacro:if>
-	<!-- <gazebo>
-		<plugin name="gazebo_ros_control" filename="libgazebo_ros_control.so">
-			<robotNamespace>mir</robotNamespace>
-			<robotParam>mir/robot_description</robotParam>
-			<controlPeriod>0.001</controlPeriod>
-			<legacyModeNS>true</legacyModeNS>
-		</plugin>
-	</gazebo>
-	 -->
-	<!-- <joint name="plattform_manipulator_joint" type="fixed">
-			<parent link="mir/base_link" />
-			<child link="ur/base_link" />
-			<origin xyz="0.215 0.1 0.35" rpy="0 0 0" />
-	</joint> -->
-	<!-- UR5 -->
-	<!-- <xacro:arg name="transmission_hw_interface" default="hardware_interface/PositionJointInterface"/> -->
-	<!-- ur5 -->
-	<!-- <xacro:include filename="$(find ur_description)/urdf/ur5.urdf.xacro" /> -->
-	<!-- arm -->
-	<!--xacro:arg name="kinematics_config" default="$(find ur_description)/config/ur5_default.yaml"/>
-	<xacro:ur5_robot prefix="ur/" joint_limited="false"
-		transmission_hw_interface="$(arg transmission_hw_interface)"
-		kinematics_file="${load_yaml('$(arg kinematics_config)')}"
-	/> -->
+    <!-- <xacro:include filename="$(find print_sim)/urdf/keyence_line_laser.gazebo.xacro" />
+    <xacro:keyence_line_laser parent_link="UR10_r/tcp" /> -->
 	<!-- <gazebo>
 		<plugin name="gazebo_ros_control" filename="libgazebo_ros_control.so">

Commit message: Add Keyence LJ-X sensor and update URDF files

File: mur/mur_description/urdf/mur_620.gazebo.xacro (robot description, xacro)
@@ -84,6 +84,6 @@
 	</joint>
 	<xacro:if value="${sim}">
-		<xacro:schunk_emh_rp_045 tf_prefix="UR10_r"	tool_link="UR10_r/flange"/>
-		<xacro:schunk_emh_rp_045 tf_prefix="UR10_l"	tool_link="UR10_l/flange"/>
+		<!-- <xacro:schunk_emh_rp_045 tf_prefix="UR10_r"	tool_link="UR10_r/flange"/>
+		<xacro:schunk_emh_rp_045 tf_prefix="UR10_l"	tool_link="UR10_l/flange"/> -->
 		<xacro:keyence_lj_x tf_prefix="UR10_r"	tool_link="UR10_r/flange"/>
 		<xacro:keyence_lj_x tf_prefix="UR10_l"	tool_link="UR10_l/flange"/>

File: tools/keyence_lj_x/urdf/keyence_lj_x.urdf.xacro (robot description, xacro)
@@ -9,5 +9,5 @@
 		</link>
 		<joint name="${tf_prefix}/gripper_joint" type="fixed">
-			<origin xyz="0 0 0.0" rpy="${-pi * 0.5} ${-pi * 0.5} ${pi}" />
+			<origin xyz="0 0 0.0" rpy="${-pi * 0.5} ${pi * 0.0} ${pi * 0.0}" />
 			<parent link="${tool_link}" />
 			<child link="${tf_prefix}/gripper" />
@@ -20,7 +20,7 @@
 			</xacro:cylinder_inertial>
 			<visual>
-				<origin xyz="0 -0.128 0" rpy="0 0 0" />
+				<origin xyz="0.05 0.05 0" rpy="0 ${pi * 0.5} ${pi * 1.0}" />
 				<geometry>
-					<mesh filename="package://schunk_emh_rp_45/meshes/visual/schunk_emh_rp_045.stl" scale="0.001 0.001 0.001"/>
+					<mesh filename="package://keyence_lj_x/meshes/visual/lj_v7200.dae" scale="1.001 1.001 1.001"/>
 				</geometry>
 				<xacro:insert_block name="material_white" />
@@ -29,5 +29,5 @@
 				<origin xyz="0 -0.128 0" rpy="0 0 0" />
 				<geometry>
-					<mesh filename="package://schunk_emh_rp_45/meshes/collision/schunk_emh_rp_045.stl" scale="0.001 0.001 0.001" />
+					<mesh filename="package://keyence_lj_x/meshes/collision/lj_v7200.stl" scale="1.001 1.001 1.001" />
 				</geometry>
 			</collision>
@@ -47,5 +47,5 @@
 		<gazebo reference="${tf_prefix}/gripper">
 			<sensor type="ray" name="line_laser">
-			<pose>0 0 0 0 0 0</pose>
+			<pose>0 0 0 1.57079632679 0 0</pose>
 			<visualize>true</visualize>
 			<update_rate>20.0</update_rate>

Commit message: Add support for different tools in URDF file

File: mur/mur_description/urdf/mur_620.gazebo.xacro (robot description, xacro)
@@ -8,4 +8,6 @@
 	<xacro:arg name="sim" default='true'/>
 	<xacro:property name="sim" value="$(arg sim)"/>
+	<xacro:arg name="tool" default='schunk_emh_rp_045'/>
+	<xacro:property name="tool" value="$(arg tool)"/>
 	<xacro:arg name="ur_l_xyz" default='0 0 0'/>
 	<xacro:arg name="ur_l_rpy" default='0 0 0'/>
@@ -84,8 +86,12 @@
 	</joint>
 	<xacro:if value="${sim}">
-		<!-- <xacro:schunk_emh_rp_045 tf_prefix="UR10_r"	tool_link="UR10_r/flange"/>
-		<xacro:schunk_emh_rp_045 tf_prefix="UR10_l"	tool_link="UR10_l/flange"/> -->
-		<xacro:keyence_lj_x tf_prefix="UR10_r"	tool_link="UR10_r/flange"/>
-		<xacro:keyence_lj_x tf_prefix="UR10_l"	tool_link="UR10_l/flange"/>
+		<xacro:if value="${tool == 'schunk_emh_rp_045'}">
+			<xacro:schunk_emh_rp_045 tf_prefix="UR10_r"	tool_link="UR10_r/flange"/>
+			<xacro:schunk_emh_rp_045 tf_prefix="UR10_l"	tool_link="UR10_l/flange"/>
+		</xacro:if>
+		<xacro:if value="${tool == 'keyence_line_laser'}">
+			<xacro:keyence_lj_x tf_prefix="UR10_r"	tool_link="UR10_r/flange"/>
+			<xacro:keyence_lj_x tf_prefix="UR10_l"	tool_link="UR10_l/flange"/>
+		</xacro:if>
 	</xacro:if>
     <!-- <xacro:include filename="$(find print_sim)/urdf/keyence_line_laser.gazebo.xacro" />
